Commit message: Added controller dependencies

File: robotiq_2f_c2_gripper_visualization/urdf/robotiq_c2_model.xacro (robot description, xacro)
@@ -5,5 +5,5 @@
  -->
 <robot name="robotiq_c2_model" xmlns:xacro="http://ros.org/wiki/xacro">
-    <xacro:include filename="$(find robotiq_2f_c2_gripper_visualization)/urdf/robotiq_c2_model_macro.xacro" />
-    <xacro:robotiq_c2_model prefix=""/>
+    <xacro:include filename="$(find robotiq_2f_c2_gripper_visualization)/urdf/robotic_c2_transmission.xacro" />
+    <xacro:robotiq_c2_model_gazebo prefix=""/>
 </robot>

File: robotiq_2f_c2_gripper_visualization/urdf/robotiq_c2_model_macro.xacro (robot description, xacro)
@@ -1,3 +1,4 @@
 <?xml version="1.0"?>
+<robot xmlns:xacro="http://ros.org/wiki/xacro">
 <!--
   robotiq_c2_model(prefix)
@@ -6,7 +7,16 @@
   there are multiple hands then a prefix followed by an "_" is needed.
 -->
-<robot xmlns:xacro="http://ros.org/wiki/xacro">
-  <xacro:macro name="robotiq_c2_model" params="prefix">
+    <xacro:macro name="default_inertial" params="mass">
+        <inertial>
+            <mass value="${mass}" />
+            <inertia ixx="1.0" ixy="0.0" ixz="0.0"
+                iyy="1.0" iyz="0.0"
+                izz="1.0" />
+        </inertial>
+    </xacro:macro>
+  <xacro:macro name="robotiq_c2_model" params="prefix transmission_hw_interface:=hardware_interface/EffortJointInterface">
+  <!-- <xacro:include filename="$(find robotiq_2f_c2_gripper_visualization)/urdf/robotic_c2_transmission.xacro"/> -->
   <link name="${prefix}robotiq_85_adapter_link">
+    <xacro:default_inertial mass="1"/>
     <visual>
       <geometry>
@@ -21,5 +31,17 @@
       <origin rpy="0 0 1.5707" xyz="0 0 0"/>
     </collision>
-  </link>
+    <inertial>
+      <origin xyz="0 0 0" rpy="0 0 0"/>
+      <mass value="7"/>
+      <inertia
+          ixx="30160574464.000000" ixy="268355824.000000" ixz="396794944.000000"
+          iyy="49449443328.00000" iyz="74363816.000000"
+          izz="47570612224.000000"/>
+    </inertial>
+  </link>
+  <gazebo reference="${prefix}robotiq_85_adapter_link">
+    <material>Gazebo/Grey</material>
+    <turnGravityOff>true</turnGravityOff>
+  </gazebo>
   <!--  /\  -->
   <joint name="${prefix}robotiq_85_base_joint" type="fixed">
@@ -31,4 +53,5 @@
   <!--  \/  -->
   <link name="${prefix}robotiq_85_base_link">
+    <xacro:default_inertial mass="1"/>
     <visual>
       <geometry>
@@ -43,5 +66,17 @@
       <origin rpy="1.5707 0 1.5707" xyz="0 0 0"/>
     </collision>
-  </link>
+    <inertial>
+      <origin xyz="0 0 0" rpy="0 0 0"/>
+      <mass value="5"/>
+      <inertia
+        ixx="29069639680.000000" ixy="16955148.000000" ixz="-75115704.000000"
+        iyy="18764271616.000000" iyz="180538688.000000"
+        izz="20780234752.000000"/>
+    </inertial>
+  </link>
+  <gazebo reference="${prefix}robotiq_85_base_link">
+    <material>Gazebo/Grey</material>
+    <turnGravityOff>true</turnGravityOff>
+  </gazebo>
   <!--  /\  -->
   <!--  /\  -->
@@ -64,4 +99,5 @@
   <!--  \/  -->
   <link name="${prefix}robotiq_85_left_knuckle_link">
+    <xacro:default_inertial mass="1"/>
     <visual>
       <geometry>
@@ -76,6 +112,19 @@
       <origin rpy="1.5707 -1.5707 0" xyz="0 .04191 -.0306"/>
     </collision>
-  </link>
+    <inertial>
+      <origin xyz="0 0 0" rpy="0 0 0"/>
+      <mass value="5"/>
+      <inertia
+        ixx="29069639680.000000" ixy="16955148.000000" ixz="-75115704.000000"
+        iyy="18764271616.000000" iyz="180538688.000000"
+        izz="20780234752.000000"/>
+    </inertial>
+  </link>
+  <gazebo reference="${prefix}robotiq_85_left_knuckle_link">
+    <material>Gazebo/Grey</material>
+    <turnGravityOff>true</turnGravityOff>
+  </gazebo>
   <link name="${prefix}robotiq_85_right_knuckle_link">
+    <xacro:default_inertial mass="1"/>
     <visual>
       <geometry>
@@ -90,5 +139,17 @@
       <origin rpy="1.5707 1.5707 0" xyz="0 .04191 -.0306"/>
     </collision>
-  </link>
+    <inertial>
+      <origin xyz="0 0 0" rpy="0 0 0"/>
+      <mass value="5"/>
+      <inertia
+        ixx="29069639680.000000" ixy="16955148.000000" ixz="-75115704.000000"
+        iyy="18764271616.000000" iyz="180538688.000000"
+        izz="20780234752.000000"/>
+    </inertial>
+  </link>
+  <gazebo reference="${prefix}robotiq_85_right_knuckle_link">
+    <material>Gazebo/Grey</material>
+    <turnGravityOff>true</turnGravityOff>
+  </gazebo>
   <!--  /\  -->
   <!--  /\  -->
@@ -110,4 +171,5 @@
   <!--  \/  -->
   <link name="${prefix}robotiq_85_left_finger_link">
+    <xacro:default_inertial mass="1"/>
     <visual>
       <geometry>
@@ -122,6 +184,19 @@
       <origin rpy="-1.5707 1.5707 0" xyz="0 -.03683 .06194"/>
     </collision>
-  </link>
+    <inertial>
+      <origin xyz="0 0 0" rpy="0 0 0"/>
+      <mass value="5"/>
+      <inertia
+        ixx="29069639680.000000" ixy="16955148.000000" ixz="-75115704.000000"
+        iyy="18764271616.000000" iyz="180538688.000000"
+        izz="20780234752.000000"/>
+    </inertial>
+  </link>
+  <gazebo reference="${prefix}robotiq_85_left_finger_link">
+    <material>Gazebo/Grey</material>
+    <turnGravityOff>true</turnGravityOff>
+  </gazebo>
   <link name="${prefix}robotiq_85_right_finger_link">
+    <xacro:default_inertial mass="1"/>
     <visual>
       <geometry>
@@ -136,5 +211,17 @@
       <origin rpy="-1.5707 -1.5707 0" xyz="0 -.03683 .06194"/>
     </collision>
-  </link>
+    <inertial>
+      <origin xyz="0 0 0" rpy="0 0 0"/>
+      <mass value="5"/>
+      <inertia
+        ixx="29069639680.000000" ixy="16955148.000000" ixz="-75115704.000000"
+        iyy="18764271616.000000" iyz="180538688.000000"
+        izz="20780234752.000000"/>
+    </inertial>
+  </link>
+  <gazebo reference="${prefix}robotiq_85_right_finger_link">
+    <material>Gazebo/Grey</material>
+    <turnGravityOff>true</turnGravityOff>
+  </gazebo>
   <!--  /\  -->
   <!--  /\  -->
@@ -158,4 +245,5 @@
   <!--  \/  -->
   <link name="${prefix}robotiq_85_left_inner_knuckle_link">
+    <xacro:default_inertial mass="1"/>
     <visual>
       <geometry>
@@ -170,6 +258,19 @@
       <origin rpy="-1.5707 1.5707 0" xyz="0 -.04843 .0127"/>
     </collision>
-  </link>
+    <inertial>
+      <origin xyz="0 0 0" rpy="0 0 0"/>
+      <mass value="5"/>
+      <inertia
+        ixx="29069639680.000000" ixy="16955148.000000" ixz="-75115704.000000"
+        iyy="18764271616.000000" iyz="180538688.000000"
+        izz="20780234752.000000"/>
+    </inertial>
+  </link>
+  <gazebo reference="${prefix}robotiq_85_left_inner_knuckle_link">
+    <material>Gazebo/Grey</material>
+    <turnGravityOff>true</turnGravityOff>
+  </gazebo>
   <link name="${prefix}robotiq_85_right_inner_knuckle_link">
+    <xacro:default_inertial mass="1"/>
     <visual>
       <geometry>
@@ -184,5 +285,17 @@
       <origin rpy="-1.5707 -1.5707 0" xyz="0 -.04843 .0127"/>
     </collision>
-  </link>
+    <inertial>
+      <origin xyz="0 0 0" rpy="0 0 0"/>
+      <mass value="5"/>
+      <inertia
+        ixx="29069639680.000000" ixy="16955148.000000" ixz="-75115704.000000"
+        iyy="18764271616.000000" iyz="180538688.000000"
+        izz="20780234752.000000"/>
+    </inertial>
+  </link>
+  <gazebo reference="${prefix}robotiq_85_right_inner_knuckle_link">
+    <material>Gazebo/Grey</material>
+    <turnGravityOff>true</turnGravityOff>
+  </gazebo>
   <!--  /\  -->
   <!--  /\  -->
@@ -206,4 +319,5 @@
   <!--  \/  -->
   <link name="${prefix}robotiq_85_left_finger_tip_link">
+    <xacro:default_inertial mass="1"/>
     <visual>
       <geometry>
@@ -218,6 +332,19 @@
       <origin rpy="-1.5707 1.5707 0" xyz="0 -.090381 .051505"/>
     </collision>
-  </link>
+    <inertial>
+      <origin xyz="0 0 0" rpy="0 0 0"/>
+      <mass value="5"/>
+      <inertia
+        ixx="29069639680.000000" ixy="16955148.000000" ixz="-75115704.000000"
+        iyy="18764271616.000000" iyz="180538688.000000"
+        izz="20780234752.000000"/>
+    </inertial>
+  </link>
+  <gazebo reference="${prefix}robotiq_85_left_finger_tip_link">
+    <material>Gazebo/Grey</material>
+    <turnGravityOff>true</turnGravityOff>
+  </gazebo>
   <link name="${prefix}robotiq_85_right_finger_tip_link">
+    <xacro:default_inertial mass="1"/>
     <visual>
       <geometry>
@@ -232,5 +359,191 @@
       <origin rpy="-1.5707 -1.5707 0" xyz="0 -.090381 .051505"/>
     </collision>
-  </link>
+    <inertial>
+      <origin xyz="0 0 0" rpy="0 0 0"/>
+      <mass value="5"/>
+      <inertia
+        ixx="29069639680.000000" ixy="16955148.000000" ixz="-75115704.000000"
+        iyy="18764271616.000000" iyz="180538688.000000"
+        izz="20780234752.000000"/>
+    </inertial>
+  </link>
+  <gazebo reference="${prefix}robotiq_85_right_finger_tip_link">
+    <material>Gazebo/Grey</material>
+    <turnGravityOff>true</turnGravityOff>
+  </gazebo>
+  <link name="world"/>
+  <!-- base_link and its fixed joint -->
+  <joint name="joint_fix" type="fixed">
+    <parent link="world"/>
+    <child link="${prefix}base_link"/>
+  </joint>
+  <link name="${prefix}base_link">
+    <collision>
+      <origin xyz="0 0 0.5" rpy="0 0 0"/>
+      <geometry>
+        <box size="0.2 0.2 0.7"/>
+      </geometry>
+    </collision>
+    <visual>
+      <origin xyz="0 0 0.5" rpy="0 0 0"/>
+      <geometry>
+        <box size="0.2 0.2 1"/>
+      </geometry>
+    </visual>
+    <inertial>
+      <origin xyz="0 0 0.5" rpy="0 0 0"/>
+      <mass value="1"/>
+      <inertia
+        ixx="1.0" ixy="0.0" ixz="0.0"
+        iyy="1.0" iyz="0.0"
+        izz="1.0"/>
+    </inertial>
+  </link>
+  <!-- link1 and its revolute joint1 relative to base_link -->
+  <!-- rotating along z axis -->
+  <joint name="${prefix}joint_a1" type="revolute">
+    <parent link="${prefix}base_link"/>
+    <child link="${prefix}link_1"/>
+    <origin xyz="0 0 1" rpy="0 0 0"/>
+    <axis xyz="0 0 1"/>
+    <limit effort="100" velocity="100" lower="-1.5708" upper="1.5708"/>
+  </joint>
+  <link name="${prefix}link_1">
+    <collision>
+      <origin xyz="0 0 0.05" rpy="0 0 0"/>
+      <geometry>
+        <cylinder length="0.1" radius="0.1"/>
+      </geometry>
+    </collision>
+    <visual>
+      <origin xyz="0 0 0.05" rpy="0 0 0"/>
+      <geometry>
+        <cylinder length="0.1" radius="0.1"/>
+      </geometry>
+    </visual>
+    <inertial>
+      <origin xyz="0 0 0.05" rpy="0 0 0"/>
+      <mass value="1"/>
+      <inertia
+        ixx="0.001" ixy="0.0" ixz="0.0"
+        iyy="0.001" iyz="0.0"
+        izz="0.001"/>
+    </inertial>
+  </link>
+  <gazebo reference="${prefix}link_1">
+    <material>Gazebo/Grey</material>
+    <turnGravityOff>true</turnGravityOff>
+  </gazebo>
+  <!-- link2 and its revolute joint2 relative to link1 -->
+  <!-- rotating along y axis -->
+  <joint name="${prefix}joint_a2" type="revolute">
+    <parent link="${prefix}link_1"/>
+    <child link="${prefix}link_2"/>
+    <origin xyz="0 0 0.1" rpy="0 0 0"/>
+    <axis xyz="0 1 0"/>
+    <limit effort="100" velocity="100" lower="-0.1" upper="1.5708"/>
+  </joint>
+  <link name="${prefix}link_2">
+    <collision>
+      <origin xyz="0 0 0.5" rpy="0 0 0"/>
+      <geometry>
+        <cylinder length="1" radius="0.1"/>
+      </geometry>
+    </collision>
+    <visual>
+      <origin xyz="0 0 0.5" rpy="0 0 0"/>
+      <geometry>
+        <cylinder length="1" radius="0.1"/>
+      </geometry>
+    </visual>
+    <inertial>
+      <origin xyz="0 0 0.5" rpy="0 0 0"/>
+      <mass value="1"/>
+      <inertia
+        ixx="0.1" ixy="0.0" ixz="0.0"
+        iyy="0.1" iyz="0.0"
+        izz="0.005"/>
+    </inertial>
+  </link>
+  <gazebo reference="${prefix}link_2">
+    <material>Gazebo/Grey</material>
+    <turnGravityOff>true</turnGravityOff>
+  </gazebo>
+  <!-- link3 and its revolute joint3 relative to link2 -->
+  <!-- rotating along y axis -->
+  <joint name="${prefix}joint_a3" type="revolute">
+    <parent link="${prefix}link_2"/>
+    <child link="${prefix}link_3"/>
+    <origin xyz="0 0 1" rpy="0 0 0"/>
+    <axis xyz="0 1 0"/>
+    <limit effort="100" velocity="100" lower="-0.1" upper="3.1416"/>
+  </joint>
+  <link name="${prefix}link_3">
+    <collision>
+      <origin xyz="0 0 0.5" rpy="0 0 0"/>
+      <geometry>
+        <cylinder length="1" radius="0.1"/>
+      </geometry>
+    </collision>
+    <visual>
+      <origin xyz="0 0 0.5" rpy="0 0 0"/>
+      <geometry>
+        <cylinder length="1" radius="0.1"/>
+      </geometry>
+    </visual>
+    <inertial>
+      <origin xyz="0 0 0.5" rpy="0 0 0"/>
+      <mass value="1"/>
+      <inertia
+        ixx="0.1" ixy="0.0" ixz="0.0"
+        iyy="0.1" iyz="0.0"
+        izz="0.005"/>
+    </inertial>
+  </link>
+  <gazebo reference="${prefix}link_3">
+    <material>Gazebo/Grey</material>
+    <turnGravityOff>true</turnGravityOff>
+  </gazebo>
+  <!-- link4 and its revolute joint4 relative to link3 -->
+  <!-- rotating along y axis -->
+  <joint name="${prefix}joint_a4" type="revolute">
+    <parent link="${prefix}link_3"/>
+    <child link="${prefix}link_4"/>
+    <origin xyz="0 0 1" rpy="0 0 0"/>
+    <axis xyz="0 1 0"/>
+    <limit effort="100" velocity="100" lower="-1.5708" upper="1.5708"/>
+  </joint>
+  <link name="${prefix}link_4">
+    <collision>
+      <origin xyz="0 0 0" rpy="1.5708 0 0"/>
+      <geometry>
+        <cylinder length="0.4" radius="0.04"/>
+      </geometry>
+    </collision>
+    <visual>
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